File: integrated-motor.kicad_sch (KiCad schematic)
At the start: 46 parts, among them J1 P_IN, J2 M01, J3 M02, J5 Programming_pins, Q1 BTN8982TA, Q2 BTN8982TA, Q3 BTN8982TA, Q4 BTN8982TA, U1 ATmega328P-P, U2 74AHC244, U3 LM22678TJ-5, U4 74AHC244

Commit message: inverse polarity protection
Parts:
- added Q6: Q_PMOS, Package_DIP:DIP-24_W7.62mm, symbol Device:Q_PMOS
- R1, R13, R14, R15, R16, R2, R3, R4: value 10k -> 1k
Connections:
- net GND: now also J5.4 (Pin_4), Q6.G; no longer J5.5 (Pin_5)
- net MOSI: now also J5.5 (Pin_5); no longer J5.2 (Pin_2)
- net P_IN+: now also Q6.S; no longer J1.1 (Pin_1)
- net RST: now also J5.3 (Pin_3); no longer J5.4 (Pin_4)
- net SCK: now also J5.2 (Pin_2); no longer J5.3 (Pin_3)
- new net: J1.1 (Pin_1), Q6.D
Other:
- moved on the sheet: C1, C10, C11, C12, C13, C14, C2, C3, C4, C5, C6, C7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
